File: Hardware/F303K8/EleMagDriver/EleMagDriver.kicad_sch (KiCad schematic)
At the start: 32 parts, among them IC1 TBD62083APG, IC2 TBD62083APG, J1 RelayA, U1 NUCLEO-F303K8

Commit message: add cad data
Parts:
- added J19, J21: Floppy_Power, Connector_PinSocket_2.54mm:PinSocket_1x04_P2.54mm_Vertical, symbol Connector:Conn_01x04_Female
- added J2: MotorDriverIn, Connector_PinHeader_2.54mm:PinHeader_1x10_P2.54mm_Vertical, symbol Connector:Conn_01x10_Female
- added J3: MotorDriveOut, Connector_PinHeader_2.54mm:PinHeader_1x06_P2.54mm_Vertical, symbol Connector:Conn_01x06_Female
- added J6: StpMotor, Connector_PinSocket_2.00mm:PinSocket_1x04_P2.00mm_Vertical, symbol Connector:Conn_01x04_Female
- C1, C2, C3, C4, C5, C6: renamed from C?; footprint (none) -> Capacitor_THT:C_Disc_D4.3mm_W1.9mm_P5.00mm
- IC1: renamed from IC?; footprint SOIC127P600X100-9N -> BD9E302EFJ-E2:SOIC127P600X100-9N
- IC2: renamed from IC?; footprint (none) -> Package_DIP:DIP-18_W7.62mm
- IC3: renamed from IC2; footprint (none) -> Package_DIP:DIP-18_W7.62mm
- IC4: renamed from IC1; footprint (none) -> Package_DIP:DIP-18_W7.62mm
- J1: renamed from J?; footprint (none) -> Connector_BarrelJack:BarrelJack_Horizontal
- J10, J11, J12, J13, J14, J15, J16, J4, J5, J8, J9: renamed from J?; footprint (none) -> Connector_PinSocket_2.00mm:PinSocket_1x02_P2.00mm_Vertical
- J17: renamed from J?; footprint (none) -> Connector_PinSocket_2.54mm:PinSocket_1x04_P2.54mm_Vertical
- J18, J20, J22: renamed from J?; footprint (none) -> Connector_PinHeader_2.54mm:PinHeader_2x17_P2.54mm_Vertical
- J7: renamed from J1; footprint (none) -> Connector_PinSocket_2.00mm:PinSocket_1x02_P2.00mm_Vertical
- L1: renamed from L?; footprint (none) -> CDRH-127NP-4R7NC:INDPM120120X800N
- R1, R2, R3: renamed from R?; footprint (none) -> Resistor_THT:R_Axial_DIN0207_L6.3mm_D2.5mm_P10.16mm_Horizontal
Connections:
- net +12V: now also J2.1 (Pin_1)
- net +5V: now also J19.1 (Pin_1), J21.1 (Pin_1)
- net GND: now also J19.2 (Pin_2), J2.3 (Pin_3), J21.2 (Pin_2), J3.3 (Pin_3), J3.4 (Pin_4)
- net Stp_A: now also J2.8 (Pin_8)
- net Stp_AN: now also J2.9 (Pin_9)
- net Stp_B: now also J2.6 (Pin_6)
- net Stp_BN: now also J2.5 (Pin_5)
- net +3.3V: now reaches U1.4_14 (+3V3)
- net +3.3V: now also J2.10 (Pin_10), J2.2 (Pin_2), J2.4 (Pin_4), J2.7 (Pin_7)
- new net Motor_OutA: J3.2 (Pin_2), J6.2 (Pin_2)
- new net Motor_OutAN: J3.1 (Pin_1), J6.1 (Pin_1)
- new net Motor_OutB: J3.6 (Pin_6), J6.3 (Pin_3)
- new net Motor_OutBN: J3.5 (Pin_5), J6.4 (Pin_4)
- no-connect marks 105 -> 108
Other:
- moved on the sheet: J17

Commit message: edit circuit
Parts:
- J10, J11, J12, J13, J14, J15, J16, J4, J5, J7, J8, J9: footprint Connector_PinSocket_2.00mm:PinSocket_1x02_P2.00mm_Vertical -> Connector_PinHeader_2.54mm:PinHeader_1x02_P2.54mm_Vertical
- J17, J19, J21: footprint Connector_PinSocket_2.54mm:PinSocket_1x04_P2.54mm_Vertical -> Connector_PinHeader_2.54mm:PinHeader_1x04_P2.54mm_Vertical
- J6: footprint Connector_PinSocket_2.00mm:PinSocket_1x04_P2.00mm_Vertical -> Connector_PinHeader_2.54mm:PinHeader_1x04_P2.54mm_Vertical

Commit message: edit circuit
Parts:
- IC1: footprint BD9E302EFJ-E2:SOIC127P600X100-9N -> (none)
- J10, J11, J12, J13, J14, J15, J16, J4, J5, J7, J8, J9: footprint Connector_PinHeader_2.54mm:PinHeader_1x02_P2.54mm_Vertical -> (none)
- J6: footprint Connector_PinHeader_2.54mm:PinHeader_1x04_P2.54mm_Vertical -> (none)
- L1: footprint CDRH-127NP-4R7NC:INDPM120120X800N -> (none)
Changed lines of the file:
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@@
       (effects (font (size 1.27 1.27)) (justify left))
     )
-    (property "Footprint" "Connector_PinHeader_2.54mm:PinHeader_1x02_P2.54mm_Vertical" (id 2) (at 139.7 67.31 0)
+    (property "Footprint" "" (id 2) (at 139.7 67.31 0)
       (effects (font (size 1.27 1.27)) hide)
     )
@@
       (effects (font (size 1.27 1.27)) (justify left))
     )
-    (property "Footprint" "Connector_PinHeader_2.54mm:PinHeader_1x02_P2.54mm_Vertical" (id 2) (at 165.1 101.6 0)
+    (property "Footprint" "" (id 2) (at 165.1 101.6 0)
       (effects (font (size 1.27 1.27)) hide)
     )
@@
       (effects (font (size 1.27 1.27)) (justify left))
     )
-    (property "Footprint" "Connector_PinHeader_2.54mm:PinHeader_1x02_P2.54mm_Vertical" (id 2) (at 165.1 116.84 0)
+    (property "Footprint" "" (id 2) (at 165.1 116.84 0)
       (effects (font (size 1.27 1.27)) hide)
     )
@@
       (effects (font (size 1.27 1.27)) (justify left))
     )
-    (property "Footprint" "Connector_PinHeader_2.54mm:PinHeader_1x02_P2.54mm_Vertical" (id 2) (at 139.7 72.39 0)
+    (property "Footprint" "" (id 2) (at 139.7 72.39 0)
       (effects (font (size 1.27 1.27)) hide)
     )
@@
       (effects (font (size 1.27 1.27)) (justify left))
     )
-    (property "Footprint" "Connector_PinHeader_2.54mm:PinHeader_1x02_P2.54mm_Vertical" (id 2) (at 165.1 106.68 0)
+    (property "Footprint" "" (id 2) (at 165.1 106.68 0)
       (effects (font (size 1.27 1.27)) hide)
     )
@@
       (effects (font (size 1.27 1.27)) (justify left))
     )
-    (property "Footprint" "Connector_PinHeader_2.54mm:PinHeader_1x02_P2.54mm_Vertical" (id 2) (at 165.1 137.16 0)
+    (property "Footprint" "" (id 2) (at 165.1 137.16 0)
       (effects (font (size 1.27 1.27)) hide)
     )
@@
       (effects (font (size 1.27 1.27)) (justify left))
     )
-    (property "Footprint" "Connector_PinHeader_2.54mm:PinHeader_1x02_P2.54mm_Vertical" (id 2) (at 165.1 121.92 0)
+    (property "Footprint" "" (id 2) (at 165.1 121.92 0)
       (effects (font (size 1.27 1.27)) hide)
     )
@@
     (property "Reference" "L1" (id 0) (at 149.86 163.83 90))
     (property "Value" "4.7u" (id 1) (at 149.86 167.64 90))
-    (property "Footprint" "CDRH-127NP-4R7NC:INDPM120120X800N" (id 2) (at 149.86 166.37 0)
+    (property "Footprint" "" (id 2) (at 149.86 166.37 0)
       (effects (font (size 1.27 1.27)) hide)
     )
@@
       (effects (font (size 1.27 1.27)) (justify left))
     )
-    (property "Footprint" "Connector_PinHeader_2.54mm:PinHeader_1x04_P2.54mm_Vertical" (id 2) (at 154.94 50.8 0)
+    (property "Footprint" "" (id 2) (at 154.94 50.8 0)
       (effects (font (size 1.27 1.27)) hide)
     )
@@
       (effects (font (size 1.27 1.27)) (justify left))
     )
-    (property "Footprint" "Connector_PinHeader_2.54mm:PinHeader_1x02_P2.54mm_Vertical" (id 2) (at 165.1 147.32 0)
+    (property "Footprint" "" (id 2) (at 165.1 147.32 0)
       (effects (font (size 1.27 1.27)) hide)
     )
@@
       (effects (font (size 1.27 1.27)) (justify left))
     )
-    (property "Footprint" "Connector_PinHeader_2.54mm:PinHeader_1x02_P2.54mm_Vertical" (id 2) (at 165.1 142.24 0)
+    (property "Footprint" "" (id 2) (at 165.1 142.24 0)
       (effects (font (size 1.27 1.27)) hide)
     )
@@
       (effects (font (size 1.27 1.27)) (justify left))
     )
-    (property "Footprint" "Connector_PinHeader_2.54mm:PinHeader_1x02_P2.54mm_Vertical" (id 2) (at 165.1 127 0)
+    (property "Footprint" "" (id 2) (at 165.1 127 0)
       (effects (font (size 1.27 1.27)) hide)
     )
@@
       (effects (font (size 1.27 1.27)) (justify left))
     )
-    (property "Footprint" "Connector_PinHeader_2.54mm:PinHeader_1x02_P2.54mm_Vertical" (id 2) (at 165.1 132.08 0)
+    (property "Footprint" "" (id 2) (at 165.1 132.08 0)
       (effects (font (size 1.27 1.27)) hide)
     )
@@
     (property "Reference" "IC1" (id 0) (at 128.27 158.75 0))
     (property "Value" "BD9E302EFJ-E2" (id 1) (at 128.27 161.29 0))
-    (property "Footprint" "BD9E302EFJ-E2:SOIC127P600X100-9N" (id 2) (at 139.7 163.83 0)
+    (property "Footprint" "" (id 2) (at 139.7 163.83 0)
       (effects (font (size 1.27 1.27)) (justify left) hide)
     )
@@
       (effects (font (size 1.27 1.27)) (justify left))
     )
-    (property "Footprint" "Connector_PinHeader_2.54mm:PinHeader_1x02_P2.54mm_Vertical" (id 2) (at 165.1 111.76 0)
+    (property "Footprint" "" (id 2) (at 165.1 111.76 0)
       (effects (font (size 1.27 1.27)) hide)
     )
@@
     )
     (path "/b367935e-06ec-4405-a687-2a6214100dc8"
-      (reference "IC1") (unit 1) (value "BD9E302EFJ-E2") (footprint "BD9E302EFJ-E2:SOIC127P600X100-9N")
+      (reference "IC1") (unit 1) (value "BD9E302EFJ-E2") (footprint "SOIC127P600X100-9N:SOIC127P600X100-9N")
     )
     (path "/23ef8a69-2f7d-4d7e-88f4-023b3c9d6b91"
@@
     )
     (path "/044d0e99-41c0-4761-bb37-20b4871c4e73"
-      (reference "J4") (unit 1) (value "SolenoidA") (footprint "Connector_PinHeader_2.54mm:PinHeader_1x02_P2.54mm_Vertical")
+      (reference "J4") (unit 1) (value "SolenoidA") (footprint "JST_B2B-XH-A(LF)(SN):JST_B2B-XH-A(LF)(SN)")
     )
     (path "/193f7a98-167c-4bb1-829a-6833e5f9344c"
-      (reference "J5") (unit 1) (value "SolenoidB") (footprint "Connector_PinHeader_2.54mm:PinHeader_1x02_P2.54mm_Vertical")
+      (reference "J5") (unit 1) (value "SolenoidB") (footprint "JST_B2B-XH-A(LF)(SN):JST_B2B-XH-A(LF)(SN)")
     )
     (path "/4a6d2edc-ec54-4d11-90f4-a3f648e57210"
-      (reference "J6") (unit 1) (value "StpMotor") (footprint "Connector_PinHeader_2.54mm:PinHeader_1x04_P2.54mm_Vertical")
+      (reference "J6") (unit 1) (value "StpMotor") (footprint "JST_B4B-XH-A(LF)(SN):JST_B4B-XH-A(LF)(SN)")
     )
     (path "/04560f96-250e-48f2-9d76-fb2d8060f360"
-      (reference "J7") (unit 1) (value "RelayA") (footprint "Connector_PinHeader_2.54mm:PinHeader_1x02_P2.54mm_Vertical")
+      (reference "J7") (unit 1) (value "RelayA") (footprint "JST_B2B-XH-A(LF)(SN):JST_B2B-XH-A(LF)(SN)")
     )
     (path "/1e9352be-f5b8-4371-a291-5cdf3774edce"
-      (reference "J8") (unit 1) (value "RelayB") (footprint "Connector_PinHeader_2.54mm:PinHeader_1x02_P2.54mm_Vertical")
+      (reference "J8") (unit 1) (value "RelayB") (footprint "JST_B2B-XH-A(LF)(SN):JST_B2B-XH-A(LF)(SN)")
     )
     (path "/d3a5f5ca-c783-4530-b6d4-2b2ad42e302b"
-      (reference "J9") (unit 1) (value "RelayC") (footprint "Connector_PinHeader_2.54mm:PinHeader_1x02_P2.54mm_Vertical")
+      (reference "J9") (unit 1) (value "RelayC") (footprint "JST_B2B-XH-A(LF)(SN):JST_B2B-XH-A(LF)(SN)")
     )
     (path "/0729df4e-3b78-4076-ac30-7047d4570e94"
-      (reference "J10") (unit 1) (value "RelayD") (footprint "Connector_PinHeader_2.54mm:PinHeader_1x02_P2.54mm_Vertical")
+      (reference "J10") (unit 1) (value "RelayD") (footprint "JST_B2B-XH-A(LF)(SN):JST_B2B-XH-A(LF)(SN)")
     )
     (path "/3c345450-fe8b-4455-b7a2-705234748c71"
-      (reference "J11") (unit 1) (value "RelayE") (footprint "Connector_PinHeader_2.54mm:PinHeader_1x02_P2.54mm_Vertical")
+      (reference "J11") (unit 1) (value "RelayE") (footprint "JST_B2B-XH-A(LF)(SN):JST_B2B-XH-A(LF)(SN)")
     )
     (path "/7cc27445-54b6-40f2-87c9-2e159a301ef8"
-      (reference "J12") (unit 1) (value "RelayF") (footprint "Connector_PinHeader_2.54mm:PinHeader_1x02_P2.54mm_Vertical")
+      (reference "J12") (unit 1) (value "RelayF") (footprint "JST_B2B-XH-A(LF)(SN):JST_B2B-XH-A(LF)(SN)")
     )
     (path "/8b1a6f89-79c8-4b8d-a254-4915a1eef869"
-      (reference "J13") (unit 1) (value "RelayG") (footprint "Connector_PinHeader_2.54mm:PinHeader_1x02_P2.54mm_Vertical")
+      (reference "J13") (unit 1) (value "RelayG") (footprint "JST_B2B-XH-A(LF)(SN):JST_B2B-XH-A(LF)(SN)")
     )
     (path "/370a9e2a-41a3-4c1d-bb4c-20160419c233"
-      (reference "J14") (unit 1) (value "RelayH") (footprint "Connector_PinHeader_2.54mm:PinHeader_1x02_P2.54mm_Vertical")
+      (reference "J14") (unit 1) (value "RelayH") (footprint "JST_B2B-XH-A(LF)(SN):JST_B2B-XH-A(LF)(SN)")
     )
     (path "/4e572461-19b9-40c4-962b-cec9997094bc"
-      (reference "J15") (unit 1) (value "RelayI") (footprint "Connector_PinHeader_2.54mm:PinHeader_1x02_P2.54mm_Vertical")
+      (reference "J15") (unit 1) (value "RelayI") (footprint "JST_B2B-XH-A(LF)(SN):JST_B2B-XH-A(LF)(SN)")
     )
     (path "/4c97cdeb-a444-4e8c-a778-02a1d5424389"
-      (reference "J16") (unit 1) (value "RelayJ") (footprint "Connector_PinHeader_2.54mm:PinHeader_1x02_P2.54mm_Vertical")
+      (reference "J16") (unit 1) (value "RelayJ") (footprint "JST_B2B-XH-A(LF)(SN):JST_B2B-XH-A(LF)(SN)")
     )
     (path "/68d75305-093c-49ea-912f-3d8fa9b557e5"
@@
     )
     (path "/47461dd1-c16a-4d87-ae8a-d300775f4d3a"
-      (reference "L1") (unit 1) (value "4.7u") (footprint "CDRH-127NP-4R7NC:INDPM120120X800N")
+      (reference "L1") (unit 1) (value "4.7u") (footprint "INDPM120120X800N:INDPM120120X800N")
     )
     (path "/d0f48553-4acb-47cd-ab26-981786651d08"

Commit message: edit circuit
Parts:
- IC1: footprint (none) -> SOIC127P600X100-9N:SOIC127P600X100-9N
- J10, J11, J12, J13, J14, J15, J16, J4, J5, J7, J8, J9: footprint (none) -> JST_B2B-XH-A(LF)(SN):JST_B2B-XH-A(LF)(SN)
- J18, J20, J22: footprint Connector_PinHeader_2.54mm:PinHeader_2x17_P2.54mm_Vertical -> SHDR34W70P254_2X17_5050X820X900P:SHDR34W70P254_2X17_5050X820X900P
- J6: footprint (none) -> JST_B4B-XH-A(LF)(SN):JST_B4B-XH-A(LF)(SN)
- L1: footprint (none) -> INDPM120120X800N:INDPM120120X800N
Changed lines of the file:
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@@
       (effects (font (size 1.27 1.27)) (justify left))
     )
-    (property "Footprint" "" (id 2) (at 139.7 67.31 0)
+    (property "Footprint" "JST_B2B-XH-A(LF)(SN):JST_B2B-XH-A(LF)(SN)" (id 2) (at 139.7 67.31 0)
       (effects (font (size 1.27 1.27)) hide)
     )
@@
       (effects (font (size 1.27 1.27)) (justify left))
     )
-    (property "Footprint" "" (id 2) (at 165.1 101.6 0)
+    (property "Footprint" "JST_B2B-XH-A(LF)(SN):JST_B2B-XH-A(LF)(SN)" (id 2) (at 165.1 101.6 0)
       (effects (font (size 1.27 1.27)) hide)
     )
@@
       (effects (font (size 1.27 1.27)) (justify left))
     )
-    (property "Footprint" "" (id 2) (at 165.1 116.84 0)
+    (property "Footprint" "JST_B2B-XH-A(LF)(SN):JST_B2B-XH-A(LF)(SN)" (id 2) (at 165.1 116.84 0)
       (effects (font (size 1.27 1.27)) hide)
     )
@@
       (effects (font (size 1.27 1.27)) (justify left))
     )
-    (property "Footprint" "" (id 2) (at 139.7 72.39 0)
+    (property "Footprint" "JST_B2B-XH-A(LF)(SN):JST_B2B-XH-A(LF)(SN)" (id 2) (at 139.7 72.39 0)
       (effects (font (size 1.27 1.27)) hide)
     )
@@
       (effects (font (size 1.27 1.27)) (justify left))
     )
-    (property "Footprint" "" (id 2) (at 165.1 106.68 0)
+    (property "Footprint" "JST_B2B-XH-A(LF)(SN):JST_B2B-XH-A(LF)(SN)" (id 2) (at 165.1 106.68 0)
       (effects (font (size 1.27 1.27)) hide)
     )
@@
       (effects (font (size 1.27 1.27)) (justify left))
     )
-    (property "Footprint" "" (id 2) (at 165.1 137.16 0)
+    (property "Footprint" "JST_B2B-XH-A(LF)(SN):JST_B2B-XH-A(LF)(SN)" (id 2) (at 165.1 137.16 0)
       (effects (font (size 1.27 1.27)) hide)
     )
@@
       (effects (font (size 1.27 1.27)) (justify left))
     )
-    (property "Footprint" "" (id 2) (at 165.1 121.92 0)
+    (property "Footprint" "JST_B2B-XH-A(LF)(SN):JST_B2B-XH-A(LF)(SN)" (id 2) (at 165.1 121.92 0)
       (effects (font (size 1.27 1.27)) hide)
     )
@@
     (property "Reference" "L1" (id 0) (at 149.86 163.83 90))
     (property "Value" "4.7u" (id 1) (at 149.86 167.64 90))
-    (property "Footprint" "" (id 2) (at 149.86 166.37 0)
+    (property "Footprint" "INDPM120120X800N:INDPM120120X800N" (id 2) (at 149.86 166.37 0)
       (effects (font (size 1.27 1.27)) hide)
     )
@@
       (effects (font (size 1.27 1.27)) (justify left))
     )
-    (property "Footprint" "" (id 2) (at 154.94 50.8 0)
+    (property "Footprint" "JST_B4B-XH-A(LF)(SN):JST_B4B-XH-A(LF)(SN)" (id 2) (at 154.94 50.8 0)
       (effects (font (size 1.27 1.27)) hide)
     )
@@
       (effects (font (size 1.27 1.27)) (justify left))
     )
-    (property "Footprint" "" (id 2) (at 165.1 147.32 0)
+    (property "Footprint" "JST_B2B-XH-A(LF)(SN):JST_B2B-XH-A(LF)(SN)" (id 2) (at 165.1 147.32 0)
       (effects (font (size 1.27 1.27)) hide)
     )
@@
       (effects (font (size 1.27 1.27)) (justify left))
     )
-    (property "Footprint" "" (id 2) (at 165.1 142.24 0)
+    (property "Footprint" "JST_B2B-XH-A(LF)(SN):JST_B2B-XH-A(LF)(SN)" (id 2) (at 165.1 142.24 0)
       (effects (font (size 1.27 1.27)) hide)
     )
@@
     (property "Reference" "J20" (id 0) (at 215.9 101.6 0))
     (property "Value" "FloppyB" (id 1) (at 215.9 104.14 0))
-    (property "Footprint" "Connector_PinHeader_2.54mm:PinHeader_2x17_P2.54mm_Vertical" (id 2) (at 214.63 128.27 0)
+    (property "Footprint" "SHDR34W70P254_2X17_5050X820X900P:SHDR34W70P254_2X17_5050X820X900P" (id 2) (at 214.63 128.27 0)
       (effects (font (size 1.27 1.27)) hide)
     )
@@
     (property "Reference" "J18" (id 0) (at 190.5 101.6 0))
     (property "Value" "FloppyA" (id 1) (at 190.5 104.14 0))
-    (property "Footprint" "Connector_PinHeader_2.54mm:PinHeader_2x17_P2.54mm_Vertical" (id 2) (at 189.23 128.27 0)
+    (property "Footprint" "SHDR34W70P254_2X17_5050X820X900P:SHDR34W70P254_2X17_5050X820X900P" (id 2) (at 189.23 128.27 0)
       (effects (font (size 1.27 1.27)) hide)
     )
@@
       (effects (font (size 1.27 1.27)) (justify left))
     )
-    (property "Footprint" "" (id 2) (at 165.1 127 0)
+    (property "Footprint" "JST_B2B-XH-A(LF)(SN):JST_B2B-XH-A(LF)(SN)" (id 2) (at 165.1 127 0)
       (effects (font (size 1.27 1.27)) hide)
     )
@@
       (effects (font (size 1.27 1.27)) (justify left))
     )
-    (property "Footprint" "" (id 2) (at 165.1 132.08 0)
+    (property "Footprint" "JST_B2B-XH-A(LF)(SN):JST_B2B-XH-A(LF)(SN)" (id 2) (at 165.1 132.08 0)
       (effects (font (size 1.27 1.27)) hide)
     )
@@
     (property "Reference" "IC1" (id 0) (at 128.27 158.75 0))
     (property "Value" "BD9E302EFJ-E2" (id 1) (at 128.27 161.29 0))
-    (property "Footprint" "" (id 2) (at 139.7 163.83 0)
+    (property "Footprint" "SOIC127P600X100-9N:SOIC127P600X100-9N" (id 2) (at 139.7 163.83 0)
       (effects (font (size 1.27 1.27)) (justify left) hide)
     )
@@
     (property "Reference" "J22" (id 0) (at 241.3 101.6 0))
     (property "Value" "FloppyC" (id 1) (at 241.3 104.14 0))
-    (property "Footprint" "Connector_PinHeader_2.54mm:PinHeader_2x17_P2.54mm_Vertical" (id 2) (at 240.03 128.27 0)
+    (property "Footprint" "SHDR34W70P254_2X17_5050X820X900P:SHDR34W70P254_2X17_5050X820X900P" (id 2) (at 240.03 128.27 0)
       (effects (font (size 1.27 1.27)) hide)
     )
@@
       (effects (font (size 1.27 1.27)) (justify left))
     )
-    (property "Footprint" "" (id 2) (at 165.1 111.76 0)
+    (property "Footprint" "JST_B2B-XH-A(LF)(SN):JST_B2B-XH-A(LF)(SN)" (id 2) (at 165.1 111.76 0)
       (effects (font (size 1.27 1.27)) hide)
     )
@@
     )
     (path "/6d94f175-8e8f-46fd-b7df-ac07f58e8223"
-      (reference "J18") (unit 1) (value "FloppyA") (footprint "Connector_PinHeader_2.54mm:PinHeader_2x17_P2.54mm_Vertical")
+      (reference "J18") (unit 1) (value "FloppyA") (footprint "SHDR34W70P254_2X17_5050X820X900P:SHDR34W70P254_2X17_5050X820X900P")
     )
     (path "/d38c51d8-ae8f-4e0d-a6fe-efc924acb4cf"
@@
     )
     (path "/619a0f06-5aa0-4b53-840d-f629b52cf5ec"
-      (reference "J20") (unit 1) (value "FloppyB") (footprint "Connector_PinHeader_2.54mm:PinHeader_2x17_P2.54mm_Vertical")
+      (reference "J20") (unit 1) (value "FloppyB") (footprint "SHDR34W70P254_2X17_5050X820X900P:SHDR34W70P254_2X17_5050X820X900P")
     )
     (path "/38dcf5fc-1b23-4014-ab21-0802283eb314"
@@
     )
     (path "/d0d06877-cb68-48ce-b520-70b71b512df7"
-      (reference "J22") (unit 1) (value "FloppyC") (footprint "Connector_PinHeader_2.54mm:PinHeader_2x17_P2.54mm_Vertical")
+      (reference "J22") (unit 1) (value "FloppyC") (footprint "SHDR34W70P254_2X17_5050X820X900P:SHDR34W70P254_2X17_5050X820X900P")
     )
     (path "/47461dd1-c16a-4d87-ae8a-d300775f4d3a"

Commit message: edit circuit
Parts:
- added R? (x5): 10k, symbol Device:R
- added R?: (no value), symbol Device:R
Connections:
- net +3.3V: no longer U1.4_14 (+3V3)
- net +5V: now also R?.1, R?.1, R?.1, R?.1, R?.1, R?.1; no longer J18.18 (Pin_18), J18.20 (Pin_20), J20.18 (Pin_18), J20.20 (Pin_20), J22.18 (Pin_18), J22.20 (Pin_20)
- net Direction1: now also IC2.5 (I5), U1.3_14 (PB5); no longer IC2.3 (I3), U1.4_8 (PA5)
- net Direction2: now also IC2.8 (I8), U1.3_7 (PB7); no longer IC2.6 (I6), U1.3_8 (PB6)
- net Direction3: now also IC3.3 (I3); no longer IC2.7 (I7)
- net GND: no longer IC4.3 (I3), IC4.4 (I4), IC4.5 (I5), J18.11 (Pin_11), J20.11 (Pin_11), J22.11 (Pin_11)
- net Relay1: now also IC3.4 (I4), IC3.5 (I5), IC3.6 (I6); no longer IC3.1 (I1), IC3.2 (I2), IC3.3 (I3)
- net Relay2: now also IC3.7 (I7), IC3.8 (I8), IC4.1 (I1); no longer IC3.4 (I4), IC3.5 (I5), IC3.6 (I6)
- net Relay3: now also IC4.2 (I2), IC4.3 (I3); no longer IC3.7 (I7), IC3.8 (I8)
- net Relay4: now also IC4.4 (I4), IC4.5 (I5); no longer IC4.1 (I1), IC4.2 (I2)
- net Step1: now also IC2.3 (I3), U1.3_15 (PB4); no longer U1.4_7 (PA6)
- net Step2: now also IC2.6 (I6), IC2.7 (I7), U1.3_8 (PB6); no longer IC2.5 (I5), U1.3_7 (PB7)
- net Step3: now also IC3.1 (I1), IC3.2 (I2); no longer IC2.8 (I8)
- net at J7.2 (Pin_2): now also IC3.15 (O4); no longer IC3.18 (O1)
- net at J10.2 (Pin_2): now also IC3.12 (O7); no longer IC3.15 (O4)
- net at J8.2 (Pin_2): now also IC3.14 (O5); no longer IC3.17 (O2)
- net at IC2.12 (O7): now also J20.12 (Pin_12); no longer J22.17 (Pin_17)
- net at IC2.14 (O5): now also J18.18 (Pin_18), R?.2; no longer J20.17 (Pin_17)
- net at IC2.15 (O4), J18.12 (Pin_12): no longer J18.19 (Pin_19)
- net at IC2.16 (O3): now also J18.20 (Pin_20), R?.2; no longer J18.17 (Pin_17)
- net at J14.2 (Pin_2): now also IC4.16 (O3); no longer IC3.11 (O8)
- net at J11.2 (Pin_2): now also IC3.11 (O8); no longer IC3.14 (O5)
- net at IC4.14 (O5): now also J16.2 (Pin_2)
- net at IC4.15 (O4): now also J15.2 (Pin_2)
- net at IC4.17 (O2): now also J13.2 (Pin_2); no longer J16.2 (Pin_2)
- net at IC4.18 (O1): now also J12.2 (Pin_2); no longer J15.2 (Pin_2)
- net at IC3.13 (O6): now also J9.2 (Pin_2); no longer J12.2 (Pin_2)
- net at IC3.16 (O3): now also J22.18 (Pin_18), R?.2; no longer J9.2 (Pin_2)
- new net: IC2.11 (O8), J20.18 (Pin_18), R?.2
- new net: IC2.13 (O6), J20.20 (Pin_20), R?.2
- new net: IC3.18 (O1), J22.20 (Pin_20), R?.2
- new net: IC3.17 (O2), J22.12 (Pin_12)
- now unconnected: J20.19 (Pin_19), J22.19 (Pin_19)
- no-connect marks 108 -> 115
Other:
- moved on the sheet: J10, J11, J12, J13, J14, J15, J16, J7, J8, J9

Commit message: edit circuit
Parts:
- R4: renamed from R?; value (none) -> 10k; footprint (none) -> Resistor_THT:R_Axial_DIN0207_L6.3mm_D2.5mm_P10.16mm_Horizontal
- R5, R6, R7, R8, R9: renamed from R?; footprint (none) -> Resistor_THT:R_Axial_DIN0207_L6.3mm_D2.5mm_P10.16mm_Horizontal
Connections:
- net +3.3V is gone; now on net +5V: J2.10 (Pin_10), J2.2 (Pin_2), J2.4 (Pin_4), J2.7 (Pin_7)

Commit message: edit circuit
Other:
- moved on the sheet: C1, C2, C3, C4, C5, C6, IC1, J1, L1, R1, R2, R3
