File: Hardware/F303K8/EleMagDriver/EleMagDriver.kicad_pcb (KiCad board)
At the start: 2 copper layers, 102.9 x 76.2 mm, 37 parts, among them IC1 BD9E302EFJ-E2, IC2 TBD62083APG, IC3 TBD62083APG, IC4 TBD62083APG, J1 Jack-DC, J10 RelayD, J11 RelayE, J12 RelayF, J13 RelayG, J14 RelayH, J15 RelayI, J16 RelayJ, J17 Floppy_Power, J18 FloppyA, J19 Floppy_Power, J2 MotorDriverIn, J20 FloppyB, J21 Floppy_Power, J22 FloppyC, J3 MotorDriveOut, J4 SolenoidA, J5 SolenoidB, J6 StpMotor, J7 RelayA, J8 RelayB, J9 RelayC, U1 NUCLEO-F303K8

Commit message: edit circuit
Parts:
- J10, J11, J12, J13, J14, J15, J16, J4, J5, J7, J8, J9: footprint Connector_PinSocket_2.00mm:PinSocket_1x02_P2.00mm_Vertical -> Connector_PinHeader_2.54mm:PinHeader_1x02_P2.54mm_Vertical
- J17, J19, J21: footprint Connector_PinSocket_2.54mm:PinSocket_1x04_P2.54mm_Vertical -> Connector_PinHeader_2.54mm:PinHeader_1x04_P2.54mm_Vertical
- J6: footprint Connector_PinSocket_2.00mm:PinSocket_1x04_P2.00mm_Vertical -> Connector_PinHeader_2.54mm:PinHeader_1x04_P2.54mm_Vertical
- moved J5 0.63 mm to (173.4, 123.8)
- moved J4 0.28 mm to (167.0, 123.8)
Routing:
- net GND: track 156.4 -> 91.2 mm, vias 1 -> 0
- net Net-(IC3-Pad16): track 88.0 -> 57.1 mm
- net Net-(IC3-Pad15): track 94.2 -> 65.0 mm, vias 1 -> 0
- net Net-(IC3-Pad18): track 68.9 -> 42.3 mm
- net +12V: track 193.9 -> 219.5 mm
- net +3.3V: track 77.3 -> 55.5 mm, vias 1 -> 0
- net Net-(IC2-Pad16): track 112.9 -> 95.2 mm
- net Net-(IC2-Pad17): track 91.3 -> 105.8 mm
- net +5V: track 239.0 -> 225.8 mm
- net Net-(IC2-Pad13): track 62.6 -> 73.0 mm
- net /Stp_BN: track 49.1 -> 59.3 mm
- net Net-(IC3-Pad14): track 83.4 -> 73.5 mm
- net Net-(IC2-Pad18): track 83.0 -> 90.3 mm
- net Net-(IC4-Pad18): track 50.3 -> 43.2 mm
- net Net-(IC2-Pad14): track 65.5 -> 72.0 mm
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
Commit message: edit circuit
Parts:
- IC1: footprint BD9E302EFJ-E2:SOIC127P600X100-9N -> SOIC127P600X100-9N:SOIC127P600X100-9N
- J10, J11, J12, J13, J14, J15, J16, J4, J5, J7, J8, J9: footprint Connector_PinHeader_2.54mm:PinHeader_1x02_P2.54mm_Vertical -> JST_B2B-XH-A(LF)(SN):JST_B2B-XH-A(LF)(SN)
- J6: footprint Connector_PinHeader_2.54mm:PinHeader_1x04_P2.54mm_Vertical -> JST_B4B-XH-A(LF)(SN):JST_B4B-XH-A(LF)(SN)
- L1: footprint CDRH-127NP-4R7NC:INDPM120120X800N -> INDPM120120X800N:INDPM120120X800N
- moved J6 5.29 mm to (172.0, 113.8), turned to 180 degrees
- moved J5 3.14 mm to (176.3, 122.7), turned to 180 degrees
- moved J4 1.31 mm to (167.6, 122.7), turned to 180 degrees
- moved J10 1.24 mm to (191.0, 60.5), turned to -90 degrees
- moved J11 1.24 mm to (197.4, 60.5), turned to -90 degrees
- moved J12 1.24 mm to (172.0, 70.6), turned to -90 degrees
- moved J15 1.24 mm to (191.0, 70.6), turned to -90 degrees
- moved J16 1.24 mm to (197.4, 70.6), turned to -90 degrees
- moved J7 1.24 mm to (172.0, 60.5), turned to -90 degrees
- moved J13 1.24 mm to (178.3, 70.6), turned to -90 degrees
- moved J14 1.24 mm to (184.7, 70.6), turned to -90 degrees
- moved J8 1.24 mm to (178.3, 60.5), turned to -90 degrees
- moved J9 1.24 mm to (184.7, 60.5), turned to -90 degrees
- moved J18 1.14 mm to (159.4, 106.2)
Routing:
- net Net-(IC2-Pad18): track 90.3 -> 86.4 mm
- net +5V: track 225.8 -> 222.6 mm
- net Net-(IC2-Pad15): track 80.2 -> 78.6 mm
- net Net-(IC2-Pad16): track 95.2 -> 94.0 mm
- net GND: track 91.2 -> 90.1 mm
- net /Motor_OutBN: track 58.4 -> 57.4 mm
- net Net-(IC2-Pad17): track 105.8 -> 105.3 mm

Commit message: edit circuit
Parts:
- J18, J20, J22: footprint Connector_PinHeader_2.54mm:PinHeader_2x17_P2.54mm_Vertical -> SHDR34W70P254_2X17_5050X820X900P:SHDR34W70P254_2X17_5050X820X900P
- moved J20 16.4 mm to (175.8, 95.4), turned to 0 degrees
- moved J18 16.4 mm to (175.7, 106.2), turned to 0 degrees
- moved J22 16.4 mm to (175.7, 84.5), turned to 0 degrees
Other:
- board size 102.9 x 76.2 mm -> 104.1 x 76.2 mm

Commit message: edit circuit
Parts:
- added R4: 10k, Resistor_THT:R_Axial_DIN0207_L6.3mm_D2.5mm_P10.16mm_Horizontal, F.Cu at (202.1, 117.3)
- added R5: 10k, Resistor_THT:R_Axial_DIN0207_L6.3mm_D2.5mm_P10.16mm_Horizontal, F.Cu at (179.2, 117.3)
- added R6: 10k, Resistor_THT:R_Axial_DIN0207_L6.3mm_D2.5mm_P10.16mm_Horizontal, F.Cu at (202.1, 105.1)
- added R7: 10k, Resistor_THT:R_Axial_DIN0207_L6.3mm_D2.5mm_P10.16mm_Horizontal, F.Cu at (199.5, 101.9)
- added R8: 10k, Resistor_THT:R_Axial_DIN0207_L6.3mm_D2.5mm_P10.16mm_Horizontal, F.Cu at (202.1, 89.8)
- added R9: 10k, Resistor_THT:R_Axial_DIN0207_L6.3mm_D2.5mm_P10.16mm_Horizontal, F.Cu at (199.5, 86.6)
- IC2, IC3, IC4: moved to B.Cu
- moved IC2 47.0 mm to (129.5, 101.6)
- moved J21 33.7 mm to (205.8, 87.6)
- moved J3 27.6 mm to (158.8, 85.7)
- moved J2 27.6 mm to (143.5, 80.6)
- moved J19 27.1 mm to (205.8, 102.9)
- moved J17 23.3 mm to (205.8, 118.1)
- moved J6 22.8 mm to (193.0, 122.6), turned to 0 degrees
- moved J11 14.3 mm to (211.5, 57.8)
- moved J16 14.3 mm to (211.5, 67.9)
- moved IC4 12.0 mm to (153.7, 74.9)
- moved J18 11.5 mm to (185.4, 112.4)
- moved J10 10.0 mm to (200.7, 57.8)
- moved J15 10.0 mm to (200.7, 67.9)
- moved J22 10.0 mm to (185.4, 81.9)
- moved J20 9.82 mm to (185.4, 97.2)
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Connections:
- IC2 pad 3: /Direction1 -> /Step1
- IC2 pad 5: /Step2 -> /Direction1
- IC2 pad 6: /Direction2 -> /Step2
- IC2 pad 7: /Direction3 -> /Step2
- IC2 pad 8: /Step3 -> /Direction2
- IC3 pad 1: /Relay1 -> /Step3
- IC3 pad 11: Net-(IC3-Pad11) -> Net-(J11-Pad2)
- IC3 pad 12: Net-(IC3-Pad12) -> Net-(J10-Pad2)
- IC3 pad 2: /Relay1 -> /Step3
- IC3 pad 3: /Relay1 -> /Direction3
- IC3 pad 4: /Relay2 -> /Relay1
- IC3 pad 5: /Relay2 -> /Relay1
- IC3 pad 6: /Relay2 -> /Relay1
- IC3 pad 7: /Relay3 -> /Relay2
- IC3 pad 8: /Relay3 -> /Relay2
- IC4 pad 1: /Relay4 -> /Relay2
- IC4 pad 14: unconnected-(IC4-Pad14) -> Net-(J16-Pad2)
- IC4 pad 15: unconnected-(IC4-Pad15) -> Net-(J15-Pad2)
- IC4 pad 16: unconnected-(IC4-Pad16) -> Net-(J14-Pad2)
- IC4 pad 17: Net-(IC4-Pad17) -> Net-(J13-Pad2)
- IC4 pad 18: Net-(IC4-Pad18) -> Net-(J12-Pad2)
- IC4 pad 2: /Relay4 -> /Relay3
- IC4 pad 3: GND -> /Relay3
- IC4 pad 4: GND -> /Relay4
- IC4 pad 5: GND -> /Relay4
- J10 pad 2: Net-(IC3-Pad15) -> Net-(J10-Pad2)
- J11 pad 2: Net-(IC3-Pad14) -> Net-(J11-Pad2)
- J12 pad 2: Net-(IC3-Pad13) -> Net-(J12-Pad2)
- J13 pad 2: Net-(IC3-Pad12) -> Net-(J13-Pad2)
- J14 pad 2: Net-(IC3-Pad11) -> Net-(J14-Pad2)
- J15 pad 2: Net-(IC4-Pad18) -> Net-(J15-Pad2)
- J16 pad 2: Net-(IC4-Pad17) -> Net-(J16-Pad2)
- J18 pad 11: GND -> unconnected-(J18-Pad11)
- J18 pad 17: Net-(IC2-Pad16) -> unconnected-(J18-Pad17)
- J18 pad 18: +5V -> Net-(IC2-Pad14)
- J18 pad 19: Net-(IC2-Pad15) -> unconnected-(J18-Pad19)
- J18 pad 20: +5V -> Net-(IC2-Pad16)
- J2 pad 10: +3.3V -> +5V
- J2 pad 2: +3.3V -> +5V
- J2 pad 4: +3.3V -> +5V
- J2 pad 7: +3.3V -> +5V
- J20 pad 11: GND -> unconnected-(J20-Pad11)
- J20 pad 12: Net-(IC2-Pad13) -> Net-(IC2-Pad12)
- J20 pad 17: Net-(IC2-Pad14) -> unconnected-(J20-Pad17)
- J20 pad 18: +5V -> Net-(IC2-Pad11)
- J20 pad 19: Net-(IC2-Pad13) -> unconnected-(J20-Pad19)
- J20 pad 20: +5V -> Net-(IC2-Pad13)
- J22 pad 11: GND -> unconnected-(J22-Pad11)
- J22 pad 12: Net-(IC2-Pad11) -> Net-(IC3-Pad17)
- J22 pad 17: Net-(IC2-Pad12) -> unconnected-(J22-Pad17)
- J22 pad 18: +5V -> Net-(IC3-Pad16)
- J22 pad 19: Net-(IC2-Pad11) -> unconnected-(J22-Pad19)
- J22 pad 20: +5V -> Net-(IC3-Pad18)
- J7 pad 2: Net-(IC3-Pad18) -> Net-(IC3-Pad15)
- J8 pad 2: Net-(IC3-Pad17) -> Net-(IC3-Pad14)
- J9 pad 2: Net-(IC3-Pad16) -> Net-(IC3-Pad13)
- U1 pad 3_14: unconnected-(U1-Pad3_14) -> /Direction1
- U1 pad 3_15: unconnected-(U1-Pad3_15) -> /Step1
- U1 pad 3_7: /Step2 -> /Direction2
- U1 pad 3_8: /Direction2 -> /Step2
- U1 pad 4_14: +3.3V -> unconnected-(U1-Pad4_14)
- U1 pad 4_7: /Step1 -> unconnected-(U1-Pad4_7)
- U1 pad 4_8: /Direction1 -> unconnected-(U1-Pad4_8)
Routing:
- net Net-(J11-Pad2): track 0.00 -> 76.0 mm
- net Net-(IC3-Pad11): track 64.5 -> 0.00 mm
- net Net-(J10-Pad2): track 0.00 -> 64.1 mm
- net +12V: track 219.9 -> 283.0 mm
- net GND: track 90.1 -> 30.6 mm
- net Net-(IC3-Pad12): track 56.0 -> 0.00 mm
- net +3.3V: track 55.5 -> 0.00 mm
- net /Relay2: track 11.2 -> 65.4 mm
- net Net-(J16-Pad2): track 0.00 -> 51.5 mm
- net Net-(IC4-Pad17): track 50.6 -> 0.00 mm
- net Net-(IC2-Pad17): track 105.3 -> 57.1 mm
- net /Stp_A: track 48.4 -> 94.6 mm
- net Net-(IC2-Pad18): track 86.4 -> 42.5 mm
- net Net-(IC4-Pad18): track 43.2 -> 0.00 mm
- net Net-(J15-Pad2): track 0.00 -> 39.6 mm
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Other:
- board size 104.1 x 76.2 mm -> 114.3 x 76.2 mm

Commit message: edit circuit
Parts:
- added G***: LOGO, LOGO:TechRing, F.Cu at (145.4, 59.1)
- added G***: LOGO, LOGO:Denken, F.Cu at (145.4, 72.4)
Routing:
- net GND: track 30.6 -> 108.8 mm
- net +12V: track 283.0 -> 265.1 mm
- net /Stp_B: track 78.5 -> 62.0 mm
- net +5V: track 187.2 -> 200.7 mm
- net /Relay2: track 65.4 -> 71.9 mm

Commit message: edit circuit
Parts:
- added REF**: MountingHole_3.2mm_M3, MountingHole:MountingHole_3.2mm_M3, F.Cu at (105.4, 123.2)
- added REF**: MountingHole_3.2mm_M3, MountingHole:MountingHole_3.2mm_M3, F.Cu at (212.1, 54.6)
- added REF**: MountingHole_3.2mm_M3, MountingHole:MountingHole_3.2mm_M3, F.Cu at (212.1, 123.2)
- added REF**: MountingHole_3.2mm_M3, MountingHole:MountingHole_3.2mm_M3, F.Cu at (105.4, 54.6)
- moved J11 4.45 mm to (211.5, 62.2)
- moved J16 3.81 mm to (211.5, 71.8)
- moved J17 0.64 mm to (205.8, 117.5)
Routing:
- net Net-(J11-Pad2): track 76.0 -> 81.2 mm
- net +12V: track 265.1 -> 268.0 mm
- net Net-(J16-Pad2): track 51.5 -> 53.1 mm

Commit message: substrate add guitar and more
Parts:
- removed C5, C6: 10u, Capacitor_THT:C_Disc_D4.3mm_W1.9mm_P5.00mm
- removed IC4: TBD62083APG, Package_DIP:DIP-18_W7.62mm
- removed L1: 4.7u, INDPM120120X800N:INDPM120120X800N
- removed R7, R8, R9: 10k, Resistor_THT:R_Axial_DIN0207_L6.3mm_D2.5mm_P10.16mm_Horizontal
- removed the REF** at (105.4, 123.2)
- removed the REF** at (212.1, 54.6)
- removed the REF** at (212.1, 123.2)
- removed the REF** at (105.4, 54.6)
- added J23: FloppyA, Connector:SHDR34W70P254_2X17_5050X820X900P, F.Cu at (158.8, 54.6)
- added J24: Floppy_Power, Connector_PinHeader_2.54mm:PinHeader_1x04_P2.54mm_Horizontal, F.Cu at (208.3, 53.3)
- added J25: FloppyB, Connector:SHDR34W70P254_2X17_5050X820X900P, F.Cu at (211.5, 80.0)
- added J26: Floppy_Power, Connector_PinHeader_2.54mm:PinHeader_1x04_P2.54mm_Horizontal, F.Cu at (208.3, 64.8)
- added REF**: MountingHole_3.2mm_M3, MountingHole:MountingHole_3.2mm_M3, F.Cu at (216.5, 125.1)
- added REF**: MountingHole_3.2mm_M3, MountingHole:MountingHole_3.2mm_M3, F.Cu at (216.5, 52.7)
- added REF**: MountingHole_3.2mm_M3, MountingHole:MountingHole_3.2mm_M3, F.Cu at (103.5, 125.1)
- added REF**: MountingHole_3.2mm_M3, MountingHole:MountingHole_3.2mm_M3, F.Cu at (103.5, 52.7)
- added RV1: 500, Potentiometer_THT:Potentiometer_Bourns_3386P_Vertical, F.Cu at (199.4, 68.6)
- added U2: NUCLEO-F303K8, Module:MODULE_NUCLEO-F303K8, F.Cu at (140.3, 76.2)
- added U3: NJM7805FA, Package_TO_SOT_THT:TO-220-3_Vertical, F.Cu at (161.2, 71.8)
- C1: footprint Capacitor_THT:C_Disc_D4.3mm_W1.9mm_P5.00mm -> Capacitor_THT:CP_Radial_D5.0mm_P2.00mm
- C2: value 0.1u -> 0.33u; footprint Capacitor_THT:C_Disc_D4.3mm_W1.9mm_P5.00mm -> Capacitor_THT:C_Disc_D4.7mm_W2.5mm_P5.00mm
- C3: footprint Capacitor_THT:C_Disc_D4.3mm_W1.9mm_P5.00mm -> Capacitor_THT:C_Disc_D4.7mm_W2.5mm_P5.00mm
- C4: value 6800p -> 100u; footprint Capacitor_THT:C_Disc_D4.3mm_W1.9mm_P5.00mm -> Capacitor_THT:CP_Radial_D6.3mm_P2.50mm
- IC1: value BD9E302EFJ-E2 -> TBD62083APG; footprint SOIC127P600X100-9N:SOIC127P600X100-9N -> Package_DIP:DIP-18_W7.62mm; moved to B.Cu
- IC2: moved to F.Cu
- J1: value Jack-DC -> MIC_{IN}; footprint Connector_BarrelJack:BarrelJack_Horizontal -> Connector_PinSocket_2.54mm:PinSocket_1x03_P2.54mm_Vertical; moved to B.Cu
- J10: value RelayD -> GuitarE; footprint JST_B2B-XH-A(LF)(SN):JST_B2B-XH-A(LF)(SN) -> Connector_JST:JST_XH_S2B-XH-A_1x02_P2.50mm_Horizontal
- J11: value RelayE -> GuitarF; footprint JST_B2B-XH-A(LF)(SN):JST_B2B-XH-A(LF)(SN) -> Connector_JST:JST_XH_S2B-XH-A_1x02_P2.50mm_Horizontal
- J12: value RelayF -> RelayA; footprint JST_B2B-XH-A(LF)(SN):JST_B2B-XH-A(LF)(SN) -> Connector_JST:JST_XH_B2B-XH-A_1x02_P2.50mm_Vertical
- J13: value RelayG -> RelayB; footprint JST_B2B-XH-A(LF)(SN):JST_B2B-XH-A(LF)(SN) -> Connector_JST:JST_XH_B2B-XH-A_1x02_P2.50mm_Vertical
- J14: value RelayH -> RelayC; footprint JST_B2B-XH-A(LF)(SN):JST_B2B-XH-A(LF)(SN) -> Connector_JST:JST_XH_B2B-XH-A_1x02_P2.50mm_Vertical
- J15: value RelayI -> RelayD; footprint JST_B2B-XH-A(LF)(SN):JST_B2B-XH-A(LF)(SN) -> Connector_JST:JST_XH_B2B-XH-A_1x02_P2.50mm_Vertical
- J16: value RelayJ -> RelayE; footprint JST_B2B-XH-A(LF)(SN):JST_B2B-XH-A(LF)(SN) -> Connector_JST:JST_XH_B2B-XH-A_1x02_P2.50mm_Vertical
- J17: value Floppy_Power -> RelayF; footprint Connector_PinHeader_2.54mm:PinHeader_1x04_P2.54mm_Vertical -> Connector_JST:JST_XH_B2B-XH-A_1x02_P2.50mm_Vertical
- J18: value FloppyA -> RelayG; footprint SHDR34W70P254_2X17_5050X820X900P:SHDR34W70P254_2X17_5050X820X900P -> Connector_JST:JST_XH_B2B-XH-A_1x02_P2.50mm_Vertical
- J19: value Floppy_Power -> RelayH; footprint Connector_PinHeader_2.54mm:PinHeader_1x04_P2.54mm_Vertical -> Connector_JST:JST_XH_B2B-XH-A_1x02_P2.50mm_Vertical
- J2: value MotorDriverIn -> LED_{OUT}; footprint Connector_PinHeader_2.54mm:PinHeader_1x10_P2.54mm_Vertical -> Connector_PinSocket_2.54mm:PinSocket_2x10_P2.54mm_Vertical
- J20: value FloppyB -> RelayI; footprint SHDR34W70P254_2X17_5050X820X900P:SHDR34W70P254_2X17_5050X820X900P -> Connector_JST:JST_XH_B2B-XH-A_1x02_P2.50mm_Vertical
- J21: value Floppy_Power -> RelayJ; footprint Connector_PinHeader_2.54mm:PinHeader_1x04_P2.54mm_Vertical -> Connector_JST:JST_XH_B2B-XH-A_1x02_P2.50mm_Vertical
- J22: value FloppyC -> Jack-DC; footprint SHDR34W70P254_2X17_5050X820X900P:SHDR34W70P254_2X17_5050X820X900P -> Connector_BarrelJack:BarrelJack_Horizontal
- J3: value MotorDriveOut -> DRV_{In}; footprint Connector_PinHeader_2.54mm:PinHeader_1x06_P2.54mm_Vertical -> Connector_PinSocket_2.54mm:PinSocket_1x08_P2.54mm_Vertical
- J4: value SolenoidA -> DRV_{OUT}; footprint JST_B2B-XH-A(LF)(SN):JST_B2B-XH-A(LF)(SN) -> Connector_PinSocket_2.54mm:PinSocket_1x08_P2.54mm_Vertical
- J5: value SolenoidB -> StpMotor; footprint JST_B2B-XH-A(LF)(SN):JST_B2B-XH-A(LF)(SN) -> Connector_JST:JST_XH_S4B-XH-A_1x04_P2.50mm_Horizontal
- J6: value StpMotor -> GuitarA; footprint JST_B4B-XH-A(LF)(SN):JST_B4B-XH-A(LF)(SN) -> Connector_JST:JST_XH_S2B-XH-A_1x02_P2.50mm_Horizontal
- J7: value RelayA -> GuitarB; footprint JST_B2B-XH-A(LF)(SN):JST_B2B-XH-A(LF)(SN) -> Connector_JST:JST_XH_S2B-XH-A_1x02_P2.50mm_Horizontal
- J8: value RelayB -> GuitarC; footprint JST_B2B-XH-A(LF)(SN):JST_B2B-XH-A(LF)(SN) -> Connector_JST:JST_XH_S2B-XH-A_1x02_P2.50mm_Horizontal
- J9: value RelayC -> GuitarD; footprint JST_B2B-XH-A(LF)(SN):JST_B2B-XH-A(LF)(SN) -> Connector_JST:JST_XH_S2B-XH-A_1x02_P2.50mm_Horizontal
- R1: value 10k -> 470
- R2: value 430k -> 1k8
- R3: value 83k -> 10k
- U1: value NUCLEO-F303K8 -> LM3914V; footprint Nucleo-f303k8:MODULE_NUCLEO-F303K8 -> Package_LCC:PLCC-20
- moved J11 118.0 mm to (107.6, 118.1)
- moved J10 106.4 mm to (107.6, 109.3)
- moved J6 98.4 mm to (107.6, 73.7), turned to -90 degrees
- moved J9 92.6 mm to (107.6, 100.3)
- moved J1 91.4 mm to (202.6, 83.9), turned to 90 degrees
- moved J8 79.0 mm to (107.6, 91.5)
- moved R1 71.7 mm to (182.9, 67.3)
- moved J22 68.2 mm to (119.4, 64.8), turned to -90 degrees
- moved C1 67.1 mm to (171.4, 73.7), turned to 180 degrees
- moved J7 65.6 mm to (107.6, 82.6)
- moved U1 64.8 mm to (181.6, 78.7), turned to -90 degrees
- moved R2 63.1 mm to (200.7, 78.7), turned to 180 degrees
- moved J15 62.6 mm to (168.9, 121.9), turned to 0 degrees
- moved C3 62.2 mm to (151.8, 59.7)
- moved R3 61.0 mm to (171.4, 62.2), turned to 0 degrees
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- renumbered G*** to G0, G*** to G1
Connections:
- C3 pad 1: Net-(C3-Pad1) -> +5V
- C3 pad 2: Net-(C3-Pad2) -> GND
- C4 pad 1: Net-(C4-Pad1) -> +12V
- C4 pad 2: Net-(C4-Pad2) -> GND
- IC1 pad 1: Net-(C3-Pad1) -> /Guitar1
- IC1 pad 2: +12V -> /Guitar2
- IC1 pad 3: +12V -> /Guitar3
- IC1 pad 4: GND -> /Guitar4
- IC1 pad 5: Net-(IC1-Pad5) -> /Guitar5
- IC1 pad 6: Net-(C4-Pad1) -> /Guitar6
- IC1 pad 8: Net-(C3-Pad2) -> GND
- IC2 pad 1: /Solenoid -> /Step1
- IC2 pad 10: +5V -> +12V
- IC2 pad 11: Net-(IC2-Pad11) -> Net-(IC2-O8)
- IC2 pad 12: Net-(IC2-Pad12) -> Net-(IC2-O7)
- IC2 pad 13: Net-(IC2-Pad13) -> Net-(IC2-O6)
- IC2 pad 14: Net-(IC2-Pad14) -> Net-(IC2-O5)
- IC2 pad 15: Net-(IC2-Pad15) -> Net-(IC2-O4)
- IC2 pad 16: Net-(IC2-Pad16) -> Net-(IC2-O3)
- IC2 pad 17: Net-(IC2-Pad17) -> Net-(IC2-O2)
- IC2 pad 18: Net-(IC2-Pad18) -> Net-(IC2-O1)
- IC2 pad 2: /Solenoid -> /Step1
- IC2 pad 3: /Step1 -> /Direction1
- IC2 pad 4: /Step1 -> /Step2
- IC2 pad 5: /Direction1 -> /Step2
- IC2 pad 6: /Step2 -> /Direction2
- IC2 pad 7: /Step2 -> /Relay1
- IC2 pad 8: /Direction2 -> /Relay1
- IC3 pad 1: /Step3 -> /Relay1
- IC3 pad 11: Net-(J11-Pad2) -> Net-(IC3-O8)
- IC3 pad 12: Net-(J10-Pad2) -> Net-(IC3-O7)
- IC3 pad 13: Net-(IC3-Pad13) -> Net-(IC3-O6)
- IC3 pad 14: Net-(IC3-Pad14) -> Net-(IC3-O5)
- IC3 pad 15: Net-(IC3-Pad15) -> Net-(IC3-O4)
- IC3 pad 16: Net-(IC3-Pad16) -> Net-(IC3-O3)
- IC3 pad 17: Net-(IC3-Pad17) -> Net-(IC3-O2)
- IC3 pad 18: Net-(IC3-Pad18) -> Net-(IC3-O1)
- IC3 pad 2: /Step3 -> /Relay2
- IC3 pad 3: /Direction3 -> /Relay2
- IC3 pad 4: /Relay1 -> /Relay2
- IC3 pad 5: /Relay1 -> /Relay3
- IC3 pad 6: /Relay1 -> /Relay3
- IC3 pad 7: /Relay2 -> /Relay4
- IC3 pad 8: /Relay2 -> /Relay4
- J1 pad 1: +12V -> +5V
- J1 pad 2: GND -> Net-(J1-Pin_2)
- J1 pad 3: (no net) -> GND
- J10 pad 2: Net-(J10-Pad2) -> Net-(IC1-O5)
- J11 pad 2: Net-(J11-Pad2) -> Net-(IC1-O6)
- J12 pad 2: Net-(J12-Pad2) -> Net-(IC2-O7)
- J13 pad 2: Net-(J13-Pad2) -> Net-(IC2-O8)
- J14 pad 2: Net-(J14-Pad2) -> Net-(IC3-O1)
- J15 pad 2: Net-(J15-Pad2) -> Net-(IC3-O2)
- J16 pad 2: Net-(J16-Pad2) -> Net-(IC3-O3)
- J17 pad 1: +5V -> +12V
- J17 pad 2: GND -> Net-(IC3-O4)
- J18 pad 1: unconnected-(J18-Pad1) -> +12V
- J18 pad 2: unconnected-(J18-Pad2) -> Net-(IC3-O5)
- J19 pad 1: +5V -> +12V
- J19 pad 2: GND -> Net-(IC3-O6)
- J2 pad 1: +12V -> Net-(J2-Pin_1)
- J2 pad 10: +5V -> +12V
- J2 pad 2: +5V -> +12V
- J2 pad 3: GND -> Net-(J2-Pin_3)
- J2 pad 4: +5V -> +12V
- J2 pad 5: /Stp_BN -> Net-(J2-Pin_5)
- J2 pad 6: /Stp_B -> +12V
- J2 pad 7: +5V -> Net-(J2-Pin_7)
- J2 pad 8: /Stp_A -> +12V
- J2 pad 9: /Stp_AN -> Net-(J2-Pin_9)
- J20 pad 1: unconnected-(J20-Pad1) -> +12V
- J20 pad 2: unconnected-(J20-Pad2) -> Net-(IC3-O7)
- J21 pad 1: +5V -> +12V
- J21 pad 2: GND -> Net-(IC3-O8)
- J22 pad 1: unconnected-(J22-Pad1) -> +12V
- J22 pad 2: unconnected-(J22-Pad2) -> GND
- J22 pad 3: unconnected-(J22-Pad3) -> (no net)
- J3 pad 1: /Motor_OutAN -> +5V
- J3 pad 2: /Motor_OutA -> GND
- J3 pad 3: GND -> +5V
- J3 pad 4: GND -> unconnected-(J3-Pin_4-Pad4)
- J3 pad 5: /Motor_OutBN -> unconnected-(J3-Pin_5-Pad5)
- J3 pad 6: /Motor_OutB -> +5V
- J4 pad 1: +5V -> +12V
- J4 pad 2: Net-(IC2-Pad18) -> GND
- J5 pad 1: +5V -> /Motor_OutB
- J5 pad 2: Net-(IC2-Pad17) -> /Motor_OutBN
- J6 pad 1: /Motor_OutAN -> +12V
- J6 pad 2: /Motor_OutA -> Net-(IC1-O1)
- J7 pad 2: Net-(IC3-Pad15) -> Net-(IC1-O2)
- J8 pad 2: Net-(IC3-Pad14) -> Net-(IC1-O3)
- J9 pad 2: Net-(IC3-Pad13) -> Net-(IC1-O4)
- R1 pad 1: Net-(C4-Pad2) -> Net-(U1-REFOUT)
- R1 pad 2: GND -> Net-(R1-Pad2)
- R2 pad 1: +5V -> Net-(R2-Pad1)
- R2 pad 2: Net-(IC1-Pad5) -> GND
- R3 pad 1: Net-(IC1-Pad5) -> +12V
- R3 pad 2: GND -> Net-(IC2-O1)
- R4 pad 1: +5V -> +12V
- R4 pad 2: Net-(IC2-Pad16) -> Net-(IC2-O3)
- R5 pad 1: +5V -> +12V
- R5 pad 2: Net-(IC2-Pad14) -> Net-(IC2-O4)
- R6 pad 1: +5V -> +12V
- R6 pad 2: Net-(IC2-Pad13) -> Net-(IC2-O6)
Routing:
- net +12V: track 268.0 -> 431.6 mm
- net GND: track 108.8 -> 0.00 mm
- net /Stp_A: track 94.9 -> 0.00 mm
- net Net-(J11-Pad2): track 81.2 -> 0.00 mm
- net Net-(IC3-Pad18): track 68.2 -> 0.00 mm
- net Net-(IC2-Pad16): track 68.2 -> 0.00 mm, vias 1 -> 0
- net Net-(IC2-Pad13): track 67.8 -> 0.00 mm
- net Net-(IC2-Pad14): track 67.8 -> 0.00 mm
- net Net-(IC2-Pad11): track 64.8 -> 0.00 mm
- net Net-(IC3-Pad16): track 64.3 -> 0.00 mm
- net Net-(J10-Pad2): track 64.1 -> 0.00 mm
- net /Stp_B: track 62.0 -> 0.00 mm
- net /Stp_AN: track 57.2 -> 0.00 mm
- net Net-(IC2-Pad17): track 57.1 -> 0.00 mm
- net Net-(IC3-Pad13): track 54.4 -> 0.00 mm
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- added copper zone on B.Cu, net GND
Other:
- board size 114.3 x 76.2 mm -> 119.4 x 78.7 mm
- board text added: "DRV8434A"
- board text removed: "TB6612"
